Commit message: Fix empty geometry in imu_link URDF — add 1cm box for visual/collision
Co-Authored-By: Claude Sonnet 4.6 <noreply@anthropic.com>

File: yahboomcar_ws/src/yahboom_description/urdf/yahboom_xgo_rviz.xacro (robot description, xacro)
@@ -826,4 +826,5 @@
         rpy="0 0 0" />
       <geometry>
+        <box size="0.01 0.01 0.01" />
       </geometry>
       <material
@@ -838,4 +839,5 @@
         rpy="0 0 0" />
       <geometry>
+        <box size="0.01 0.01 0.01" />
       </geometry>
     </collision>

Commit message: Fix action interruption and URDF standing height
yahboom_ctrl: don't call stop() while an action is playing — the browser
publishes zero cmd_vel on key release which was cutting actions short.
The lock clears as soon as the user sends intentional movement, or on reset.

URDF: raise base_footprint→base_link from 10mm to 108mm (default standing
height). The previous value was a CAD residual that put the body in the ground.

Co-Authored-By: Claude Sonnet 4.6 <noreply@anthropic.com>

File: yahboomcar_ws/src/yahboom_description/urdf/yahboom_xgo_rviz.xacro (robot description, xacro)
@@ -9,5 +9,5 @@
     <parent link="base_footprint"/>
     <child link="base_link" />
-    <origin xyz="0 0 0.010" rpy="0 0 0"/>
+    <origin xyz="0 0 0.108" rpy="0 0 0"/>
   </joint>
   <link

Commit message: Simplify to single nav mode, remove robot mode, fix IMU cube
- run_jazzy.sh: --nav is now the default, --robot removed
- entrypoint_nav.sh: map is optional — Nav2 skipped if no map,
  teleop + LiDAR + rf2o always run
- Dockerfile: default ENTRYPOINT is now entrypoint_nav.sh
- entrypoint.sh removed
- yahboom_ctrl: remove dead-reckoning odom (rf2o provides real odom)
- URDF: remove imu_link visual/collision (was showing as floating cube)

Co-Authored-By: Claude Sonnet 4.6 <noreply@anthropic.com>

File: yahboomcar_ws/src/yahboom_description/urdf/yahboom_xgo_rviz.xacro (robot description, xacro)
@@ -821,25 +821,4 @@
         izz="4.25931212063486E-06" />
     </inertial>
-    <visual>
-      <origin
-        xyz="0 0 0"
-        rpy="0 0 0" />
-      <geometry>
-        <box size="0.01 0.01 0.01" />
-      </geometry>
-      <material
-        name="">
-        <color
-          rgba="1 1 1 1" />
-      </material>
-    </visual>
-    <collision>
-      <origin
-        xyz="0 0 0"
-        rpy="0 0 0" />
-      <geometry>
-        <box size="0.01 0.01 0.01" />
-      </geometry>
-    </collision>
   </link>
   <joint

Commit message: align TF stack on base_link (VM reference)
- urdf: remove base_footprint→base_link wrapper — base_link is now root,
  avoiding TF conflict when rf2o publishes odom→base_link
- ekf_robot.yaml: base_link_frame: base_link
- entrypoints: rf2o base_frame_id=base_link on all three modes;
  apply same ros2 run + init_pose_from_topic fix to entrypoint_robot
- slam_toolbox_params.yaml: new config with base_frame=base_link,
  transform_timeout=0.5s, wired into entrypoint_slam
- README: update TF tree diagram

Co-Authored-By: Claude Sonnet 4.6 <noreply@anthropic.com>

File: yahboomcar_ws/src/yahboom_description/urdf/yahboom_xgo_rviz.xacro (robot description, xacro)
@@ -5,10 +5,4 @@
 <robot name="xgo" xmlns:xacro="http://ros.org/wiki/xacro">
   <xacro:property name="pi"  value  = "3.14"/>
-  <link name="base_footprint"/>
-  <joint name="base_joint" type="fixed">
-    <parent link="base_footprint"/>
-    <child link="base_link" />
-    <origin xyz="0 0 0.108" rpy="0 0 0"/>
-  </joint>
   <link
     name="base_link">

File: yahboomcar_ws/src/yahboom_description/urdf/yahboom_xgo_rviz_local.xacro (robot description, xacro)
@@ -5,10 +5,4 @@
 <robot name="xgo" xmlns:xacro="http://ros.org/wiki/xacro">
   <xacro:property name="pi"  value  = "3.14"/>
-  <link name="base_footprint"/>
-  <joint name="base_joint" type="fixed">
-    <parent link="base_footprint"/>
-    <child link="base_link" />
-    <origin xyz="0 0 0.010" rpy="0 0 0"/>
-  </joint>
   <link
     name="base_link">

Commit message: urdf: restore base_footprint→base_link, align nav stack on base_footprint
Correct TF architecture: odom→base_footprint (rf2o/EKF) + fixed URDF
joint base_footprint→base_link at +0.108 m (robot_state_publisher).
No TF conflict, KDL warning gone, robot visual correct in RViz2.

- yahboom_xgo_rviz.xacro: add base_footprint link + fixed joint 0.108 m
- yahboom_xgo_rviz_local.xacro: same at 0.010 m
- rf2o_params.yaml: base_frame_id → base_footprint
- ekf_robot.yaml: base_link_frame → base_footprint
- slam_toolbox_params.yaml: base_frame → base_footprint
- nav2_params.yaml: AMCL base_frame_id → base_footprint
- yahboom_ctrl.py: dead-reckoning child_frame_id → base_footprint
- laser_Patrol_xgo_RS200.py: base_frame → base_footprint

Co-Authored-By: Claude Sonnet 4.6 <noreply@anthropic.com>

File: yahboomcar_ws/src/yahboom_description/urdf/yahboom_xgo_rviz.xacro (robot description, xacro)
@@ -5,4 +5,10 @@
 <robot name="xgo" xmlns:xacro="http://ros.org/wiki/xacro">
   <xacro:property name="pi"  value  = "3.14"/>
+  <link name="base_footprint"/>
+  <joint name="base_joint" type="fixed">
+    <parent link="base_footprint"/>
+    <child link="base_link"/>
+    <origin xyz="0 0 0.108" rpy="0 0 0"/>
+  </joint>
   <link
     name="base_link">

File: yahboomcar_ws/src/yahboom_description/urdf/yahboom_xgo_rviz_local.xacro (robot description, xacro)
@@ -5,4 +5,10 @@
 <robot name="xgo" xmlns:xacro="http://ros.org/wiki/xacro">
   <xacro:property name="pi"  value  = "3.14"/>
+  <link name="base_footprint"/>
+  <joint name="base_joint" type="fixed">
+    <parent link="base_footprint"/>
+    <child link="base_link"/>
+    <origin xyz="0 0 0.010" rpy="0 0 0"/>
+  </joint>
   <link
     name="base_link">
